File: PCB/Cherry_MX_Keyboard_PCB.sch (KiCad schematic (older format))
At the start: 33 parts, among them SW1 MX_1, SW10 MX_7, SW11 MX_11, SW12 MX_15, SW13 MX_4, SW14 MX_8, SW15 MX_12, SW16 MX_16, SW2 MX_5, SW3 MX_9, SW4 MX_13, SW5 MX_2, SW6 MX_6, SW7 MX_10, SW8 MX_14, SW9 MX_3, U1 ARDUINO_PRO_MICRO

Commit message: keyboard PCB V 0.2
Parts:
- R1, R10, R11, R12, R13, R14, R15, R16, R2, R3, R4, R5, R6, R7, R8, R9: footprint R:R4 -> Cherry_MX_Keyboard:R4
- U1: footprint arduino_pro_micro:ARDUINO_PRO_MICRO -> Cherry_MX_Keyboard:ARDUINO_PRO_MICRO
Changed lines of the file:
@@
 F 0 "R2" H 1150 4300 50  0000 C CNN
 F 1 "10K" H 1150 4400 50  0000 C CNN
-F 2 "R:R4" H 1150 4350 60  0001 C CNN
+F 2 "Cherry_MX_Keyboard:R4" H 1150 4350 60  0001 C CNN
 F 3 "" H 1150 4350 60  0000 C CNN
 	1    1150 4350
@@
 F 0 "R3" H 1150 5050 50  0000 C CNN
 F 1 "10K" H 1150 5150 50  0000 C CNN
-F 2 "R:R4" H 1150 5100 60  0001 C CNN
+F 2 "Cherry_MX_Keyboard:R4" H 1150 5100 60  0001 C CNN
 F 3 "" H 1150 5100 60  0000 C CNN
 	1    1150 5100
@@
 F 0 "R4" H 1150 5750 50  0000 C CNN
 F 1 "10K" H 1150 5850 50  0000 C CNN
-F 2 "R:R4" H 1150 5800 60  0001 C CNN
+F 2 "Cherry_MX_Keyboard:R4" H 1150 5800 60  0001 C CNN
 F 3 "" H 1150 5800 60  0000 C CNN
 	1    1150 5800
@@
 F 0 "R1" H 1150 3750 50  0000 C CNN
 F 1 "10K" H 1150 3850 50  0000 C CNN
-F 2 "R:R4" H 1150 3800 60  0001 C CNN
+F 2 "Cherry_MX_Keyboard:R4" H 1150 3800 60  0001 C CNN
 F 3 "" H 1150 3800 60  0000 C CNN
 	1    1150 3800
@@
 F 0 "R6" H 2650 4300 50  0000 C CNN
 F 1 "10K" H 2650 4400 50  0000 C CNN
-F 2 "R:R4" H 2650 4350 60  0001 C CNN
+F 2 "Cherry_MX_Keyboard:R4" H 2650 4350 60  0001 C CNN
 F 3 "" H 2650 4350 60  0000 C CNN
 	1    2650 4350
@@
 F 0 "R7" H 2650 5050 50  0000 C CNN
 F 1 "10K" H 2650 5150 50  0000 C CNN
-F 2 "R:R4" H 2650 5100 60  0001 C CNN
+F 2 "Cherry_MX_Keyboard:R4" H 2650 5100 60  0001 C CNN
 F 3 "" H 2650 5100 60  0000 C CNN
 	1    2650 5100
@@
 F 0 "R8" H 2650 5750 50  0000 C CNN
 F 1 "10K" H 2650 5850 50  0000 C CNN
-F 2 "R:R4" H 2650 5800 60  0001 C CNN
+F 2 "Cherry_MX_Keyboard:R4" H 2650 5800 60  0001 C CNN
 F 3 "" H 2650 5800 60  0000 C CNN
 	1    2650 5800
@@
 F 0 "R5" H 2650 3750 50  0000 C CNN
 F 1 "10K" H 2650 3850 50  0000 C CNN
-F 2 "R:R4" H 2650 3800 60  0001 C CNN
+F 2 "Cherry_MX_Keyboard:R4" H 2650 3800 60  0001 C CNN
 F 3 "" H 2650 3800 60  0000 C CNN
 	1    2650 3800
@@
 F 0 "R10" H 4100 4300 50  0000 C CNN
 F 1 "10K" H 4100 4400 50  0000 C CNN
-F 2 "R:R4" H 4100 4350 60  0001 C CNN
+F 2 "Cherry_MX_Keyboard:R4" H 4100 4350 60  0001 C CNN
 F 3 "" H 4100 4350 60  0000 C CNN
 	1    4100 4350
@@
 F 0 "R11" H 4100 5050 50  0000 C CNN
 F 1 "10K" H 4100 5150 50  0000 C CNN
-F 2 "R:R4" H 4100 5100 60  0001 C CNN
+F 2 "Cherry_MX_Keyboard:R4" H 4100 5100 60  0001 C CNN
 F 3 "" H 4100 5100 60  0000 C CNN
 	1    4100 5100
@@
 F 0 "R12" H 4100 5750 50  0000 C CNN
 F 1 "10K" H 4100 5850 50  0000 C CNN
-F 2 "R:R4" H 4100 5800 60  0001 C CNN
+F 2 "Cherry_MX_Keyboard:R4" H 4100 5800 60  0001 C CNN
 F 3 "" H 4100 5800 60  0000 C CNN
 	1    4100 5800
@@
 F 0 "R9" H 4100 3750 50  0000 C CNN
 F 1 "10K" H 4100 3850 50  0000 C CNN
-F 2 "R:R4" H 4100 3800 60  0001 C CNN
+F 2 "Cherry_MX_Keyboard:R4" H 4100 3800 60  0001 C CNN
 F 3 "" H 4100 3800 60  0000 C CNN
 	1    4100 3800
@@
 F 0 "R14" H 5650 4300 50  0000 C CNN
 F 1 "10K" H 5650 4400 50  0000 C CNN
-F 2 "R:R4" H 5650 4350 60  0001 C CNN
+F 2 "Cherry_MX_Keyboard:R4" H 5650 4350 60  0001 C CNN
 F 3 "" H 5650 4350 60  0000 C CNN
 	1    5650 4350
@@
 F 0 "R15" H 5650 5050 50  0000 C CNN
 F 1 "10K" H 5650 5150 50  0000 C CNN
-F 2 "R:R4" H 5650 5100 60  0001 C CNN
+F 2 "Cherry_MX_Keyboard:R4" H 5650 5100 60  0001 C CNN
 F 3 "" H 5650 5100 60  0000 C CNN
 	1    5650 5100
@@
 F 0 "R16" H 5650 5750 50  0000 C CNN
 F 1 "10K" H 5650 5850 50  0000 C CNN
-F 2 "R:R4" H 5650 5800 60  0001 C CNN
+F 2 "Cherry_MX_Keyboard:R4" H 5650 5800 60  0001 C CNN
 F 3 "" H 5650 5800 60  0000 C CNN
 	1    5650 5800
@@
 F 0 "R13" H 5650 3750 50  0000 C CNN
 F 1 "10K" H 5650 3850 50  0000 C CNN
-F 2 "R:R4" H 5650 3800 60  0001 C CNN
+F 2 "Cherry_MX_Keyboard:R4" H 5650 3800 60  0001 C CNN
 F 3 "" H 5650 3800 60  0000 C CNN
 	1    5650 3800
@@
 F 0 "U1" V 8750 3500 60  0000 C CNN
 F 1 "ARDUINO_PRO_MICRO" V 8650 3500 60  0000 C CNN
-F 2 "arduino_pro_micro:ARDUINO_PRO_MICRO" H 8500 4050 60  0001 C CNN
+F 2 "Cherry_MX_Keyboard:ARDUINO_PRO_MICRO" H 8500 4050 60  0001 C CNN
 F 3 "" H 8500 4050 60  0000 C CNN
 	1    8650 3550
@@
 R_SW
 $Comp
-L +3V3 #PWR?
+L +3V3 #PWR010
 U 1 1 59905579
 P 7400 3000
-F 0 "#PWR?" H 7400 2850 50  0001 C CNN
+F 0 "#PWR010" H 7400 2850 50  0001 C CNN
 F 1 "+3V3" H 7400 3140 50  0000 C CNN
 F 2 "" H 7400 3000 50  0000 C CNN
